File: PecanFemto3.sch (EAGLE design)
At the start: 50 parts, among them IC1 SPV1040T, IC3 EVA7M, IC4 SI4060/3, IC5 LPC824M201JHI33E, U1 TPS62203DBVT

Commit message: Changed part values
Parts:
- R6: value 22k -> 10k
- U1: value TPS62203DBVT -> TPS62205DBVT
Changed lines of the file:
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@@
 <attribute name="OC_NEWARK" value="unknown"/>
 </part>
-<part name="U1" library="TPS62203" deviceset="TPS62203DBVT" device="">
+<part name="U1" library="TPS62203" deviceset="TPS62203DBVT" device="" value="TPS62205DBVT">
 <attribute name="MF" value="TEXAS INSTRUMENTS"/>
 </part>
@@
 <part name="SUPPLY11" library="SparkFun-Aesthetics" deviceset="VCC" device=""/>
 <part name="GND13" library="SparkFun-Aesthetics" deviceset="GND" device=""/>
-<part name="R6" library="PecanPico6" deviceset="RES-0402" device="" value="22k">
+<part name="R6" library="PecanPico6" deviceset="RES-0402" device="" value="10k">
 <attribute name="MF" value=""/>
 <attribute name="MPN" value=""/>

Commit message: Fixed PecanPico3 errors Removed paste from large pads Added pullup to RADIO_SDN Fixed TCXO swapping (pins inverted) Updated Designators (on silkscreen layer)
Parts:
- added R8: 22k, PecanPico6:RES-0402
- U$1: value TXC 7Z-26.000MCG-T -> TXC_7Z; OC_NEWARK unknown -> (none)
- renumbered TCXO to U$1
Connections:
- net RADIO_SDN: now also R8.1
- net VCC: now also R8.2
Changed lines of the file:
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@@
-<attribute name="OC_NEWARK" value="unknown"/>
-</part>
-<part name="TCXO" library="tcxo" deviceset="TXC_7Z" device="" value="TXC 7Z-26.000MCG-T">
-<attribute name="MF" value=""/>
-<attribute name="MPN" value=""/>
 <attribute name="OC_NEWARK" value="unknown"/>
 </part>
@@
 </part>
 <part name="GND32" library="SparkFun-Aesthetics" deviceset="GND" device=""/>
+<part name="U$1" library="tcxo" deviceset="TXC_7Z" device=""/>
+<part name="R8" library="PecanPico6" deviceset="RES-0402" device="" value="22k">
+<attribute name="MF" value=""/>
+<attribute name="MPN" value=""/>
+<attribute name="OC_NEWARK" value="unknown"/>
+</part>
+<part name="SUPPLY5" library="SparkFun-Aesthetics" deviceset="VCC" device=""/>
 </parts>
 <sheets>
@@
 <attribute name="MPN" x="162.56" y="-26.67" size="1.778" layer="96" display="off"/>
 </instance>
-<instance part="TCXO" gate="TCXO" x="182.88" y="-27.94">
-<attribute name="OC_NEWARK" x="182.88" y="-27.94" size="1.778" layer="96" display="off"/>
-<attribute name="MF" x="182.88" y="-27.94" size="1.778" layer="96" display="off"/>
-<attribute name="MPN" x="182.88" y="-27.94" size="1.778" layer="96" display="off"/>
-</instance>
 <instance part="VBAT" gate="1" x="58.42" y="119.38">
 <attribute name="OC_NEWARK" x="58.42" y="119.38" size="1.778" layer="96" display="off"/>
@@
 </instance>
 <instance part="GND32" gate="1" x="66.04" y="78.74"/>
+<instance part="U$1" gate="TCXO" x="182.88" y="-27.94"/>
+<instance part="R8" gate="G$1" x="271.78" y="33.02" rot="R90">
+<attribute name="OC_NEWARK" x="271.78" y="33.02" size="1.778" layer="96" display="off"/>
+<attribute name="MF" x="271.78" y="33.02" size="1.778" layer="96" display="off"/>
+<attribute name="MPN" x="271.78" y="33.02" size="1.778" layer="96" display="off"/>
+</instance>
+<instance part="SUPPLY5" gate="G$1" x="271.78" y="40.64"/>
 </instances>
 <busses>
@@
 <wire x1="162.56" y1="-31.75" x2="162.56" y2="-33.02" width="0.1524" layer="91"/>
 <junction x="162.56" y="-33.02"/>
-<pinref part="TCXO" gate="TCXO" pin="GND"/>
+<pinref part="U$1" gate="TCXO" pin="GND"/>
 </segment>
 <segment>
@@
 <pinref part="GND22" gate="1" pin="GND"/>
 <wire x1="200.66" y1="-33.02" x2="200.66" y2="-38.1" width="0.1524" layer="91"/>
-<pinref part="TCXO" gate="TCXO" pin="AFC"/>
+<pinref part="U$1" gate="TCXO" pin="AFC"/>
 </segment>
 <segment>
@@
 <wire x1="317.5" y1="10.16" x2="317.5" y2="7.62" width="0.1524" layer="91"/>
 </segment>
+<segment>
+<pinref part="R8" gate="G$1" pin="2"/>
+<pinref part="SUPPLY5" gate="G$1" pin="VCC"/>
+<wire x1="271.78" y1="38.1" x2="271.78" y2="40.64" width="0.1524" layer="91"/>
+</segment>
 </net>
 <net name="CS_RADIO" class="0">
@@
 <segment>
 <pinref part="IC4" gate="G$1" pin="1_SDN"/>
-<wire x1="264.16" y1="25.4" x2="266.7" y2="25.4" width="0.1524" layer="91"/>
-<label x="266.7" y="25.4" size="1.27" layer="95" xref="yes"/>
+<wire x1="264.16" y1="25.4" x2="271.78" y2="25.4" width="0.1524" layer="91"/>
+<label x="279.4" y="25.4" size="1.27" layer="95" xref="yes"/>
+<pinref part="R8" gate="G$1" pin="1"/>
+<wire x1="271.78" y1="25.4" x2="279.4" y2="25.4" width="0.1524" layer="91"/>
+<wire x1="271.78" y1="27.94" x2="271.78" y2="25.4" width="0.1524" layer="91"/>
+<junction x="271.78" y="25.4"/>
 </segment>
 <segment>
@@
 <pinref part="C6" gate="G$1" pin="1"/>
 <wire x1="203.2" y1="-22.86" x2="203.2" y2="-17.78" width="0.1524" layer="91"/>
-<pinref part="TCXO" gate="TCXO" pin="OUT"/>
 <wire x1="203.2" y1="-22.86" x2="210.82" y2="-22.86" width="0.1524" layer="91"/>
 <junction x="203.2" y="-22.86"/>
 <pinref part="C7" gate="G$1" pin="1"/>
 <wire x1="210.82" y1="-22.86" x2="210.82" y2="-17.78" width="0.1524" layer="91"/>
+<pinref part="U$1" gate="TCXO" pin="OUT"/>
 </segment>
 </net>
@@
 <pinref part="C5" gate="G$1" pin="2"/>
 <wire x1="162.56" y1="-24.13" x2="162.56" y2="-22.86" width="0.1524" layer="91"/>
-<pinref part="TCXO" gate="TCXO" pin="VCC"/>
 <wire x1="162.56" y1="-22.86" x2="162.56" y2="-20.32" width="0.1524" layer="91"/>
 <junction x="162.56" y="-22.86"/>
 <label x="162.56" y="-20.32" size="1.27" layer="95" rot="R90" xref="yes"/>
-</segment>
-</net>
+<pinref part="U$1" gate="TCXO" pin="VCC"/>
+</segment>
+</net>

Commit message: Changed TCXO designator, improved EVA7M package
Parts:
- IC6: value TXC_7Z -> KT2016K26000BCW18ZAS
- renumbered U$1 to IC6, U1 to IC2
Changed lines of the file:
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@@
 <attribute name="OC_NEWARK" value="unknown"/>
 </part>
-<part name="U1" library="TPS62203" deviceset="TPS62203DBVT" device="" value="TPS62205DBVT">
+<part name="IC2" library="TPS62203" deviceset="TPS62203DBVT" device="" value="TPS62205DBVT">
 <attribute name="MF" value="TEXAS INSTRUMENTS"/>
 </part>
@@
 </part>
 <part name="GND32" library="SparkFun-Aesthetics" deviceset="GND" device=""/>
-<part name="U$1" library="tcxo" deviceset="TXC_7Z" device=""/>
+<part name="IC6" library="tcxo" deviceset="TXC_7Z" device="" value="KT2016K26000BCW18ZAS"/>
 <part name="R8" library="PecanPico6" deviceset="RES-0402" device="" value="22k">
 <attribute name="MF" value=""/>
@@
 <instance part="GND11" gate="1" x="340.36" y="30.48"/>
 <instance part="GND9" gate="1" x="350.52" y="-35.56"/>
-<instance part="GND22" gate="1" x="200.66" y="-40.64"/>
+<instance part="GND22" gate="1" x="205.74" y="-40.64"/>
 <instance part="L3" gate="G$1" x="134.62" y="111.76">
 <attribute name="OC_NEWARK" x="134.62" y="111.76" size="1.778" layer="96" display="off"/>
@@
 <attribute name="MPN" x="210.82" y="-12.7" size="1.778" layer="96" display="off"/>
 </instance>
-<instance part="U1" gate="A" x="109.22" y="106.68">
+<instance part="IC2" gate="A" x="109.22" y="106.68">
 <attribute name="MF" x="109.22" y="106.68" size="1.778" layer="96" display="off"/>
 </instance>
@@
 </instance>
 <instance part="GND32" gate="1" x="66.04" y="78.74"/>
-<instance part="U$1" gate="TCXO" x="182.88" y="-27.94"/>
+<instance part="IC6" gate="TCXO" x="182.88" y="-27.94"/>
 <instance part="R8" gate="G$1" x="271.78" y="33.02" rot="R90">
 <attribute name="OC_NEWARK" x="271.78" y="33.02" size="1.778" layer="96" display="off"/>
@@
 <wire x1="162.56" y1="-31.75" x2="162.56" y2="-33.02" width="0.1524" layer="91"/>
 <junction x="162.56" y="-33.02"/>
-<pinref part="U$1" gate="TCXO" pin="GND"/>
+<pinref part="IC6" gate="TCXO" pin="GND"/>
 </segment>
 <segment>
@@
 </segment>
 <segment>
-<wire x1="198.12" y1="-33.02" x2="200.66" y2="-33.02" width="0.1524" layer="91"/>
+<wire x1="198.12" y1="-33.02" x2="205.74" y2="-33.02" width="0.1524" layer="91"/>
 <pinref part="GND22" gate="1" pin="GND"/>
-<wire x1="200.66" y1="-33.02" x2="200.66" y2="-38.1" width="0.1524" layer="91"/>
-<pinref part="U$1" gate="TCXO" pin="AFC"/>
+<wire x1="205.74" y1="-33.02" x2="205.74" y2="-38.1" width="0.1524" layer="91"/>
+<pinref part="IC6" gate="TCXO" pin="AFC"/>
 </segment>
 <segment>
@@
 <wire x1="88.9" y1="96.52" x2="88.9" y2="81.28" width="0.1524" layer="91"/>
 <pinref part="GND17" gate="1" pin="GND"/>
-<pinref part="U1" gate="A" pin="GND"/>
+<pinref part="IC2" gate="A" pin="GND"/>
 </segment>
 <segment>
@@
 <wire x1="147.32" y1="111.76" x2="152.4" y2="111.76" width="0.1524" layer="91"/>
 <pinref part="SUPPLY2" gate="G$1" pin="VCC"/>
-<pinref part="U1" gate="A" pin="FB"/>
+<pinref part="IC2" gate="A" pin="FB"/>
 </segment>
 <segment>
@@
 <pinref part="C7" gate="G$1" pin="1"/>
 <wire x1="210.82" y1="-22.86" x2="210.82" y2="-17.78" width="0.1524" layer="91"/>
-<pinref part="U$1" gate="TCXO" pin="OUT"/>
+<pinref part="IC6" gate="TCXO" pin="OUT"/>
 </segment>
 </net>
@@
 <pinref part="VBAT" gate="1" pin="P"/>
 <wire x1="60.96" y1="119.38" x2="66.04" y2="119.38" width="0.1524" layer="91"/>
-<pinref part="U1" gate="A" pin="EN"/>
-<pinref part="U1" gate="A" pin="VI"/>
+<pinref part="IC2" gate="A" pin="EN"/>
+<pinref part="IC2" gate="A" pin="VI"/>
 <pinref part="R6" gate="G$1" pin="2"/>
 <wire x1="66.04" y1="109.22" x2="66.04" y2="111.76" width="0.1524" layer="91"/>
@@
 <pinref part="L3" gate="G$1" pin="1"/>
 <wire x1="129.54" y1="111.76" x2="127" y2="111.76" width="0.1524" layer="91"/>
-<pinref part="U1" gate="A" pin="SW"/>
+<pinref part="IC2" gate="A" pin="SW"/>
 </segment>
 </net>
@@
 <junction x="162.56" y="-22.86"/>
 <label x="162.56" y="-20.32" size="1.27" layer="95" rot="R90" xref="yes"/>
-<pinref part="U$1" gate="TCXO" pin="VCC"/>
-</segment>
-</net>
+<pinref part="IC6" gate="TCXO" pin="VCC"/>
+</segment>
+</net>
